Commit message: rename megarover_samples to kaitpv

File: urdf/body/body.urdf.xacro (robot description, xacro)
@@ -11,5 +11,5 @@
         <origin xyz="-0.028241 -0.073553 0.01"/>
         <geometry>
-          <mesh filename="package://megarover_samples/meshes/dae/megarover.dae"/>
+          <mesh filename="package://kaitpv/meshes/dae/megarover.dae"/>
           <!--<mesh filename="$(find kobuki_description)/meshes/main_body.dae"/>-->
           <!--<mesh filename="/home/rover/3d/megarover.dae"/>-->

File: urdf/body/vbody.urdf.xacro (robot description, xacro)
@@ -1,5 +1,5 @@
 <?xml version="1.0"?>
 <robot xmlns:xacro="http://ros.org/wiki/xacro">
-  <xacro:include filename="$(find megarover_samples)/urdf/body/body.gazebo.xacro"/>
+  <xacro:include filename="$(find kaitpv)/urdf/body/body.gazebo.xacro"/>
   <xacro:macro name="base_v0" params="parent *joint_origin">
     <joint name="base_link_joint" type="fixed">
@@ -11,10 +11,10 @@
       <visual>
         <geometry>
-          <mesh filename="package://megarover_samples/meshes/dae/vmega_body.dae"/>
+          <mesh filename="package://kaitpv/meshes/dae/vmega_body.dae"/>
         </geometry>
       </visual>
       <collision>
         <geometry>
-          <mesh filename="package://megarover_samples/meshes/stl/vmega_body.stl"/>
+          <mesh filename="package://kaitpv/meshes/stl/vmega_body.stl"/>
         </geometry>
       </collision>

File: urdf/wheel/vwheel.urdf.xacro (robot description, xacro)
@@ -1,7 +1,7 @@
 <?xml version="1.0"?>
 <robot xmlns:xacro="http://ros.org/wiki/xacro">
-  <xacro:include filename="$(find megarover_samples)/urdf/common.xacro"/>
-  <xacro:include filename="$(find megarover_samples)/urdf/wheel/wheel.transmission.xacro"/>
-  <xacro:include filename="$(find megarover_samples)/urdf/wheel/wheel.gazebo.xacro"/>
+  <xacro:include filename="$(find kaitpv)/urdf/common.xacro"/>
+  <xacro:include filename="$(find kaitpv)/urdf/wheel/wheel.transmission.xacro"/>
+  <xacro:include filename="$(find kaitpv)/urdf/wheel/wheel.gazebo.xacro"/>
   <xacro:property name="wheel_radius" value="0.076"/>
   <xacro:property name="wheel_length" value="0.03"/>
@@ -17,5 +17,5 @@
       <visual>
         <geometry>
-          <mesh filename="package://megarover_samples/meshes/dae/vmega_wheel.dae"/>
+          <mesh filename="package://kaitpv/meshes/dae/vmega_wheel.dae"/>
         </geometry>
       </visual>
