Commit message: fix world

File: robots/vmegarover.urdf.xacro (robot description, xacro)
@@ -8,5 +8,5 @@
   <link name="base_footprint"/>
   <xacro:base_v0 parent="base_footprint">
-    <origin xyz="-1.4 1.4 0"/>
+    <origin xyz="0 0 0"/>
   </xacro:base_v0>
   <!-- Wheel -->

Commit message: add ped actors

File: robots/vmegarover.urdf.xacro (robot description, xacro)
@@ -23,5 +23,5 @@
   <!-- Front LRF -->
   <xacro:lrf_v0 prefix="front" parent="base_link">
-    <origin xyz="0.099 0 0.1015"/>
+    <origin xyz="0.099 0 0.9"/>
   </xacro:lrf_v0>
   <!-- Front LRF Upper-->

Commit message: add rviz for vo

File: robots/vmegarover.urdf.xacro (robot description, xacro)
@@ -23,5 +23,5 @@
   <!-- Front LRF -->
   <xacro:lrf_v0 prefix="front" parent="base_link">
-    <origin xyz="0.099 0 0.9"/>
+    <origin xyz="0.099 0 0.5"/>
   </xacro:lrf_v0>
   <!-- Front LRF Upper-->

File: urdf/lrf/lrf.gazebo.xacro (robot description, xacro)
@@ -6,5 +6,5 @@
         <pose>0 0 0 0 0 0</pose>
         <visualize>true</visualize>
-        <update_rate>40</update_rate>
+        <update_rate>10</update_rate>
         <ray>
           <scan>
